File: Reliable_Controller_For_Railworks/Schematics/SELE_PROJECT.brd (EAGLE design)
At the start: 160 x 100 mm, 31 parts, among them IC1 D1 (24LC1025), IC2 D2 (7812L), IC3 D3 (7805L), IC4 VN460SP, IC5 VN460SP, T1 230V to 12V AC, U1 328P, U2 LTC485N, X1 16MHz, X3 LAMP CONNECTOR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

Commit message: Minor bug fix and implementation of log printing in a server command
Other:
- board size 160 x 100 mm -> 68.6 x 79.7 mm

Commit message: Finish
Finish Project
Connections:
- net N$14: now also T1.2
Changed lines of the file:
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@@
 <drawing>
 <settings>
-<setting alwaysvectorfont="yes"/>
+<setting alwaysvectorfont="no"/>
 <setting verticaltext="up"/>
 </settings>
@@
 <classes>
 <class number="0" name="default" width="50.8" drill="0.0381">
-<clearance class="0" value="0.0254"/>
 </class>
 </classes>
@@
 <wire x1="33.6804" y1="14.0208" x2="33.72" y2="13.97" width="0.1524" layer="1"/>
 <wire x1="11.43" y1="43.1292" x2="11.43" y2="43.18" width="0.1524" layer="1"/>
+<contactref element="T1" pad="2"/>
 </signal>
 </signals>
